File: hardware/tail_board/tail_board.kicad_pcb (KiCad board)
At the start: 2 copper layers, 68 x 68 mm, 18 parts, among them J1 DC IN, J2 DC THRU, J3 Head, J4 Camera, J5 8P8C_Shielded, Q1 DMP3037LSS-13

Commit message: V1 of the tailboard
Parts:
- added ?: , Graphics, F.Cu at (105.8, 126.8)
- added ?: , Graphics, F.Cu at (119.5, 98.3)
- added ?: , Graphics, F.Cu at (156.0, 122.1)
- added ?: , Graphics, F.Cu at (146.5, 98.3)
- added ?: , Graphics, F.Cu at (162.8, 101.8)
- added ?: , Graphics, F.Cu at (133.5, 123.1)
- added ?: , Graphics, F.Cu at (119.0, 102.6)
- added ?: , Graphics, F.Cu at (92.5, 98.3)
- added ?: , Graphics, F.Cu at (92.0, 102.6)
- added ?: , Graphics, F.Cu at (156.0, 111.1)
- added ?: , Graphics, F.Cu at (146.8, 136.1)
- added C2: 100u, Capacitor_SMD:CP_Elec_6.3x9.9, F.Cu at (147.5, 122.1)
- added C3: 100u, Capacitor_SMD:CP_Elec_6.3x9.9, F.Cu at (147.5, 114.1)
- added J6: Bottom camera, winterbloom:USB_B_Receptacle_Horizontal, F.Cu at (91.2, 94.7)
- added J7: Bottom camera, Connector_JST:JST_SH_SM04B-SRSS-TB_1x04-1MP_P1.00mm_Horizontal, F.Cu at (92.5, 142.6)
- J1, J2: footprint winterbloom:TerminalBlock_4UCON_1x02_P3.50mm_Horizontal -> winterbloom:TerminalBlock_CUI_TB002-500_1x02_P5.00mm_Vertical
- J4: value Camera -> Top camera; footprint Connector_USB:USB_B_Lumberg_2411_02_Horizontal -> winterbloom:USB_B_Receptacle_Horizontal
- Je: renamed from J3; footprint Connector_USB:USB_B_Lumberg_2411_02_Horizontal -> winterbloom:USB_B_Receptacle_Horizontal
- R1, R2, R3: footprint Resistor_SMD:R_0603_1608Metric_Pad0.98x0.95mm_HandSolder -> winterbloom:R_0402_HandSolder
- moved J1 88.6 mm to (162.8, 122.1), turned to 90 degrees
- moved J2 87.4 mm to (162.8, 111.1), turned to 90 degrees
- moved D1 84.6 mm to (146.5, 144.3)
- moved R1 79.4 mm to (146.5, 142.1)
- moved Q1 78.3 mm to (162.5, 132.1), turned to 90 degrees
- moved D2 78.0 mm to (157.5, 83.1)
- moved R2 78.0 mm to (157.5, 88.1), turned to -90 degrees
- moved F1 68.5 mm to (152.5, 141.1)
- moved Je 56.0 mm to (145.2, 94.7)
- moved C1 48.5 mm to (147.5, 106.1), turned to 0 degrees
- moved H3 30.0 mm to (163.5, 83.1)
- moved H4 30.0 mm to (163.5, 143.1)
- moved J5 29.9 mm to (133.4, 136.1)
- moved J4 3.03 mm to (118.2, 94.7)
- moved D3 2.28 mm to (130.5, 83.1)
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Connections:
- H1 pad 1: GND -> unconnected-(H1-Pad1)
- H2 pad 1: GND -> unconnected-(H2-Pad1)
- J5 pad 1: +24V -> /CAM_D+
- J5 pad 2: +24V -> /CAM_D-
- J5 pad 4: GND -> /HEAD_D+
- J5 pad 6: /HEAD_D+ -> +24V
- J5 pad 7: /CAM_D- -> GND
- J5 pad 8: /CAM_D+ -> +24V
Routing:
- net /BTM_CAM_D+: track 0.00 -> 49.1 mm
- net /BTM_CAM_D-: track 0.00 -> 46.9 mm
- net Net-(J6-Pad1): track 0.00 -> 46.0 mm
- net +VDC: track 31.3 -> 0.00 mm
- net +24V: track 45.5 -> 15.7 mm
- net /HEAD_D-: track 63.7 -> 40.7 mm
- net /HEAD_D+: track 62.1 -> 41.0 mm
- net Net-(F1-Pad1): track 15.8 -> 0.00 mm
- net /CAM_D-: track 42.5 -> 37.0 mm
- net Net-(D1-Pad1): track 6.81 -> 2.56 mm
- net Net-(D3-Pad1): track 6.26 -> 9.00 mm
- net /HEAD_VBUS: track 21.8 -> 23.9 mm
- net /CAM_VBUS: track 25.1 -> 23.5 mm
- net /CAM_D+: track 42.9 -> 41.4 mm
- net Net-(D2-Pad1): track 8.62 -> 7.59 mm
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- added copper zone on F.Cu, net +24V
- added copper zone on F.Cu, net +VDC
- added copper zone on F.Cu, net Net-(F1-Pad1)
- added copper zone on B.Cu, net Net-(J6-Pad4)
- added copper zone on F.Cu, net Net-(J6-Pad4)
Other:
- board size 68 x 68 mm -> 98 x 68 mm
- board text added: "${TITLE} ${REVISION} ${ISSUE_DATE} ${COMMENT1} ${COMMENT2} ${COMMENT3} ${COMMENT4}"
- board text added: "PCB Specifications: - 2 copper layers - Size: 98 x 68 mm - Thickness: 1.6 mm - Material: FR4 TG-140+ - Min track width/spacing: 0.153 mm (5 mil) - Min hole size: 0.3 mm - Soldermask: Pink/Purple/Matte Black - Silkscreen: Black/White - Finish: ENIG 2U{dblquote} - Copper: 1 oz - UL Marking: on bottom silkscreen"
- board text removed: "+ -"
- board text removed: "BOARD"
- board text removed: "CAMERA"
- board text removed: "HEAD"
- board text removed: "PCB Specifications: - 2 copper layers - Size: 100 x 30 mm - Thickness: 1.6 mm - Material: FR4 TG-140+ - Min track width/spacing: 0.153 mm (5 mil) - Min hole size: 0.3 mm - Soldermask: Pink/Purple/Matte Black - Silkscreen: Black/White - Finish: ENIG 2U{dblquote} - Copper: 1 oz - UL Marking: on bottom silkscreen"
