File: hardware/jellyfish_tailboard/jellyfish_tailboard.kicad_pcb (KiCad board)
At the start: 2 copper layers, 98 x 68 mm, 33 parts, among them J1 DC IN, J2 DC THRU, J4 Top camera, J5 8P8C_Shielded, J6 Bottom camera, J7 Bottom camera, Q1 DMP3037LSS-13

Commit message: touchup tailboard
Parts:
- removed the ? at (105.8, 126.8)
- removed the ? at (162.8, 101.8)
- removed the ? at (119.0, 102.6)
- removed the ? at (92.0, 102.6)
- removed the ? at (146.8, 136.1)
- added ?: , Graphics, F.Cu at (119.5, 102.9)
- added ?: , Graphics, F.Cu at (105.9, 122.5)
- added ?: , Graphics, F.Cu at (162.8, 101.5)
- added ?: , Graphics, F.Cu at (148.1, 129.4)
- added ?: , Graphics, F.Cu at (120.2, 140.8)
- added ?: , Graphics, F.Cu at (92.5, 102.9)
- added ?: , Graphics, F.Cu at (92.5, 138.2)
- added D4: SMAJ28A, winterbloom:D_SMA, F.Cu at (159.4, 135.6)
- added D5: PDZ16BGWJ, winterbloom:D_SOD-123, F.Cu at (148.5, 140.8)
- added R4: 47k, winterbloom:R_0402_HandSolder, F.Cu at (147.8, 144.8)
- R1: value 5.1k -> 5K1
- moved F1 14.9 mm to (163.5, 131.1), turned to 180 degrees
- moved Q1 11.4 mm to (155.5, 141.1), turned to 0 degrees
- moved D1 4.10 mm to (144.0, 141.1), turned to 90 degrees
- moved R1 3.40 mm to (144.5, 144.8)
- moved C1 1.05 mm to (147.5, 105.0)
- moved C2 1.05 mm to (147.5, 121.0)
- moved C3 1.05 mm to (147.5, 113.0)
- renumbered Je to J3
Connections:
- F1 pad 1: Net-(F1-Pad1) -> +VDC
- F1 pad 2: +24V -> /post fuse
- Q1 pad 1: Net-(F1-Pad1) -> +24V
- Q1 pad 2: Net-(F1-Pad1) -> +24V
- Q1 pad 3: Net-(F1-Pad1) -> +24V
- Q1 pad 4: GND -> /gate
- Q1 pad 5: +VDC -> /post fuse
- Q1 pad 6: +VDC -> /post fuse
- Q1 pad 7: +VDC -> /post fuse
- Q1 pad 8: +VDC -> /post fuse
Routing:
- net +24V: track 15.7 -> 0.00 mm
- net /gate: track 0.00 -> 7.17 mm
- net /CAM_D-: track 37.0 -> 41.4 mm
- net /BTM_CAM_D-: track 46.9 -> 49.2 mm
- added copper zone on F.Cu, net /post fuse
- removed copper zone on F.Cu, net Net-(F1-Pad1)
