File: hardware/jellyfish_tailboard/jellyfish_tailboard.kicad_sch (KiCad schematic)
At the start: 22 parts, among them J1 DC IN, J2 DC THRU, J3 Head, J4 Top camera, J5 8P8C_Shielded, J6 Bottom camera, J7 Bottom camera, Q1 DMP3037LSS-13

Commit message: touchup tailboard
Parts:
- added D4: SMAJ28A, winterbloom:D_SMA, symbol Device:D_Zener_Filled
- added D5: PDZ16BGWJ, winterbloom:D_SOD-123, symbol Device:D_Zener_Filled
- added R4: 47k, winterbloom:R_0402_HandSolder, symbol Device:R_US
- C1, C2, C3: Rating (none) -> 50V
- F1: Rating (none) -> 3A
- R1: value 5.1k -> 5K1
Connections:
- net +24V: now also Q1.1 (S), Q1.2 (S), Q1.3 (S), D5.1 (K); no longer F1.2
- net +VDC: now also F1.1; no longer Q1.5 (D), Q1.6 (D), Q1.7 (D), Q1.8 (D)
- net GND: now also D4.2 (A), R4.2; no longer Q1.4 (G)
- new net gate: D5.2 (A), Q1.4 (G), R4.1
- new net post fuse: D4.1 (K), F1.2, Q1.5 (D), Q1.6 (D), Q1.7 (D), Q1.8 (D)
Other:
- note removed: "TODO: Use CUI footprint"
- moved on the sheet: C1, C2, C3, D1, D2, D3, F1, J3, J4, J5, J6, J7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
