File: hardware/jellyfish/jellyfish.kicad_sch (KiCad schematic)
At the start: 3 parts

Commit message: Update license on all hardware files
Other:
- title: Candela Head -> Jellyfish
Changed lines of the file:
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@@
   (paper "USLetter")
   (title_block
-    (title "Candela Head")
-    (date "2022-07-27")
+    (title "Jellyfish")
+    (date "2022-10-14")
     (rev "v1")
     (company "Winterbloom")
     (comment 1 "Alethea Flowers")
-    (comment 2 "CERN-OHL-P V2")
+    (comment 2 "CERN-OHL-S V2")
   )
   (junction (at 121.92 186.69) (diameter 0) (color 0 0 0 0)
